File: KICAD Workspace/Licenta_Vlad/_autosave-BLDC inverter.kicad_pcb (KiCad board)
At the start: 2 copper layers, 130.8 x 107.7 mm, 103 parts, among them J1 Conn_01x03, J2 Conn_01x02, J3 Conn_01x03, J4 Conn_01x02, J5 Conn_01x03, J6 Conn_01x03, Q1 BC547, Q2 IRF9530, U1 IR2101, U10 LP2950-3.3_TO92, U2 IR2101, U3 IR2101, U4 L7805, U5 LM2576HVT-12, U6 LM2576HVT-12, U7 ACS754, U8 LM393, U9 LM393

Commit message: PCB version 1 after big big failure .......................
Parts:
- removed 0.1uF1: C_Small, Capacitor_THT:CP_Radial_D8.0mm_P3.50mm
- added J7: Conn_01x03, Connector_PinHeader_2.54mm:PinHeader_1x03_P2.54mm_Vertical, F.Cu at (35.3, 122.3)
- moved R31 237.5 mm to (39.4, 153.8), turned to 90 degrees
- moved R29 195.4 mm to (55.6, 137.7), turned to 270 degrees
- moved C7 182.2 mm to (97.9, 112.3), turned to 90 degrees
- moved Q1 177.5 mm to (64.5, 140.0), turned to 270 degrees
- moved C1 177.3 mm to (100.2, 124.2), turned to 90 degrees
- moved R32 176.7 mm to (45.8, 138.4), turned to 270 degrees
- moved C9 174.9 mm to (97.9, 142.1), turned to 90 degrees
- moved C3 167.5 mm to (97.8, 150.6), turned to 270 degrees
- moved R30 161.9 mm to (50.9, 106.3), turned to 270 degrees
- moved C2 161.7 mm to (67.8, 89.3), turned to 180 degrees
- moved C12 158.8 mm to (108.6, 138.7), turned to 270 degrees
- moved R6 157.7 mm to (117.2, 146.4)
- moved Q2 155.1 mm to (39.4, 114.3), turned to 90 degrees
- moved C10 152.8 mm to (108.8, 108.8), turned to 270 degrees
- moved C19 142.4 mm to (161.9, 152.1)
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Connections:
- C30 pad 1: Net-(C30-Pad1) -> /Sheet5CB00087/3V3
- R15 pad 1: Net-(R15-Pad1) -> /Sheet5CB00087/PHASE_C
- R28 pad 1: Net-(C30-Pad1) -> /Sheet5CB00087/3V3
- U10 pad 1: Net-(C30-Pad1) -> /Sheet5CB00087/3V3
- U7 pad 1: +5V -> /Sheet5CB00087/3V3
Routing:
- net GNDREF: track 303.7 -> 1103.6 mm, vias 0 -> 2
- net /Sheet5CB00087/CP: track 0.00 -> 272.6 mm
- net /Sheet5CB00087/5V: track 13.8 -> 197.4 mm
- net /Sheet5CB00087/PHASE_A: track 0.00 -> 174.6 mm
- net /Sheet5CB00087/12V_Bootstrap: track 60.6 -> 232.3 mm
- net /Sheet5CB00087/PHASE_B: track 0.00 -> 163.4 mm
- net /Sheet5CB00087/PHASE_C: track 0.00 -> 159.6 mm
- net /Sheet5CB00087/BEMF_C: track 0.00 -> 157.6 mm
- net /Sheet5CB00087/CURRENT_SENSOR: track 0.00 -> 150.3 mm
- net /Sheet5CB00087/3V3: track 0.00 -> 149.2 mm
- net /Sheet5CB00087/BEMF_B: track 0.00 -> 142.2 mm
- net /Sheet5CB00087/EXTIB: track 0.00 -> 129.6 mm
- net /Sheet5CB00087/BEMF_A: track 0.00 -> 124.3 mm
- net /Sheet5CB00087/EXTIC: track 0.00 -> 113.8 mm
- net /Sheet5CB00087/BEMF_REF: track 0.00 -> 113.3 mm
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- added copper zone on B.Cu, net GNDREF
- added copper zone on F.Cu, net GNDREF
Other:
- board size 130.8 x 107.7 mm -> 259.7 x 159.5 mm
- board text added: "BACIU VLAD EUSEBIU"
- board text added: "SENSORLESS MOTOR CONTROLLER"
