File: KICAD Workspace/OnlyInverter/OnlyInverter.kicad_pcb (KiCad board)
At the start: 2 copper layers, 264.2 x 170.8 mm, 87 parts, among them J1 Conn_01x03, J2 Conn_01x03, J3 Conn_01x03, J4 Conn_01x03, J5 Conn_01x02, J6 Conn_01x03, J7 Conn_01x02, Q1 BC547, Q2 IRF9530, U1 L7805, U2 ACS754, U3 LP2950-3.3_TO92, U4 IR2101, U5 IR2101, U6 IR2101, U7 LM393, U8 LM393

Commit message: Added SMD version of ESC.
Parts:
- added D11: 1N5819, Diode_THT:D_DO-41_SOD81_P10.16mm_Horizontal, F.Cu at (188.0, 48.8)
- added D12: 1N5819, Diode_THT:D_DO-41_SOD81_P10.16mm_Horizontal, F.Cu at (188.1, 68.7)
- added D13: 1N5819, Diode_THT:D_DO-41_SOD81_P10.16mm_Horizontal, F.Cu at (182.0, 86.6)
- added D14: 1N5819, Diode_THT:D_DO-41_SOD81_P10.16mm_Horizontal, F.Cu at (182.2, 103.9)
- added D15: 1N5819, Diode_THT:D_DO-41_SOD81_P10.16mm_Horizontal, F.Cu at (182.2, 118.9)
- added D16: 1N5819, Diode_THT:D_DO-41_SOD81_P10.16mm_Horizontal, F.Cu at (181.9, 143.3)
- added R25: 10K, Resistor_THT:R_Axial_DIN0411_L9.9mm_D3.6mm_P15.24mm_Horizontal, F.Cu at (148.8, 51.7)
- added R26: 10K, Resistor_THT:R_Axial_DIN0411_L9.9mm_D3.6mm_P15.24mm_Horizontal, F.Cu at (142.2, 91.6)
- added R27: 10K, Resistor_THT:R_Axial_DIN0411_L9.9mm_D3.6mm_P15.24mm_Horizontal, F.Cu at (145.4, 129.2)
- R13, R14, R15: value 150k -> 10K
- moved J6 25.2 mm to (271.0, 44.7)
- moved Q2 6.67 mm to (65.3, 135.8), turned to 90 degrees
- moved C18 5.84 mm to (195.7, 41.8)
- moved C19 5.84 mm to (195.7, 55.4)
- moved R28 5.84 mm to (238.5, 26.2)
- moved R29 5.84 mm to (233.6, 26.0)
- moved R30 5.84 mm to (228.9, 26.2)
- moved U7 5.84 mm to (220.0, 46.6)
- moved U8 5.84 mm to (212.3, 52.5)
- moved C17 1.14 mm to (140.1, 130.9)
Connections:
- Q2 pad 2: /V_BAT+ -> Net-(Q2-Pad2)
- Q2 pad 3: Net-(Q2-Pad3) -> /V_BAT+
- R4 pad 1: Net-(Q2-Pad3) -> Net-(Q2-Pad2)
Routing:
- net GNDREF: track 1291.1 -> 1268.3 mm
- net /EXTIB: track 38.1 -> 60.1 mm
- net /EXTIC: track 48.0 -> 69.3 mm
- net /EXTIA: track 46.1 -> 67.2 mm
- net Net-(Q2-Pad3): track 10.5 -> 0.00 mm
- net Net-(Q2-Pad2): track 0.00 -> 10.5 mm
- net /BEMF_B: track 128.9 -> 120.2 mm
- net Net-(D9-Pad2): track 31.2 -> 38.7 mm
- net /BEMF_REF: track 158.4 -> 152.6 mm
- net /BEMF_C: track 134.9 -> 129.1 mm
- net /BEMF_A: track 97.4 -> 91.6 mm
- net /PHASE_A: track 220.0 -> 225.0 mm
- net /PHASE_C: track 170.9 -> 175.7 mm
- net Net-(D5-Pad2): track 36.0 -> 40.8 mm
- net /PHASE_B: track 184.5 -> 189.0 mm
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- removed copper zone on F.Cu, net GNDREF
Other:
- board size 264.2 x 170.8 mm -> 262.6 x 168.5 mm
