File: KICAD Workspace/OnlyInverter/OnlyInverter.sch (KiCad schematic (older format))
At the start: 87 parts, among them J1 Conn_01x03, J2 Conn_01x03, J3 Conn_01x03, J4 Conn_01x03, J5 Conn_01x02, J6 Conn_01x03, J7 Conn_01x02, Q1 BC547, Q2 IRF9530, U1 L7805, U2 ACS754, U3 LP2950-3.3_TO92, U4 IR2101, U5 IR2101, U6 IR2101, U7 LM393, U8 LM393

Commit message: Added SMD version of ESC.
Parts:
- removed Q2: IRF9530, Package_TO_SOT_THT:TO-220-3_Vertical, symbol Transistor_FET:IRF3205
- added D11, D12, D13, D14, D15, D16: 1N5819, Diode_THT:D_DO-41_SOD81_P10.16mm_Horizontal, symbol Diode:1N5819
- added Q2: IRF9530, Package_TO_SOT_THT:TO-220-3_Vertical, symbol Transistor_FET:IRF9540N
- added R25, R26, R27: 10K, Resistor_THT:R_Axial_DIN0411_L9.9mm_D3.6mm_P15.24mm_Horizontal, symbol Device:R
- R13, R14, R15: value 150k -> 10K
Connections:
- wire segments 336 -> 381
